File: hw/hwv0/hwv0.sch (KiCad schematic (older format))
At the start: 28 parts, among them J1 AVR-ISP-6, SW1 SW_Push, U1 ATtiny84A-MU, U2 LCD_1602, U3 MAX232I

Commit message: Yet to add sensors and ICSP connections
Parts:
- added J3: RS232, Connector_Dsub:DSUB-9_Female_Horizontal_P2.77x2.84mm_EdgePinOffset4.94mm_Housed_MountingHolesOffset7.48mm, symbol Connector:DB9_Female_MountingHoles
- R2: value 10K -> 270
- U4: renamed from U?; footprint (none) -> Package_TO_SOT_SMD:SOT-223-3_TabPin2
- gave numbers to parts that had none: 10
Connections:
- wire segments 88 -> 95
Other:
- note added: "CONNECTORS\n"
- note added: "PRESSURE SENSOR\n"
- note added: "RS232_CONN\n"

Commit message: Almost completed PCB
Connections:
- wire segments 95 -> 97
Changed lines of the file:
@@
 Wire Wire Line
 	2300 2000 2500 2000
-Wire Wire Line
-	2500 2100 2300 2100
 Text Label 2500 2000 0    50   ~ 0
 STRAINGAUGE+
@@
 Text Notes 1100 5850 0    100  ~ 0
 CONNECTORS\n
+Text Label 4700 2200 0    50   ~ 0
+MISO
+Text Label 4700 2300 0    50   ~ 0
+MOSI
+Wire Wire Line
+	4500 2200 4700 2200
+Connection ~ 4500 2200
+Wire Wire Line
+	4700 2300 4400 2300
+Connection ~ 4400 2300
+Wire Wire Line
+	2300 2100 4700 2100
+Text Label 4700 2100 0    50   ~ 0
+SCK
 $EndSCHEMATC

Commit message: finished PCB
Other:
- note added: "Data Acquisition System\n"
Changed lines of the file:
@@
 Text Label 4700 2100 0    50   ~ 0
 SCK
+Text Notes 7350 7500 0    79   ~ 0
+Data Acquisition System\n
 $EndSCHEMATC

Commit message: made schematic more clear
Parts:
- removed StrainGauge1: Conn_01x04_Female, Connector_JST:JST_XH_B04B-XH-AM_1x04_P2.50mm_Vertical, symbol Connector:Conn_01x04_Female
- added StrainGauge1: Conn_01x04_Shielded, Connector_JST:JST_XH_B05B-XH-A_1x05_P2.50mm_Vertical, symbol Connector_Generic_Shielded:Conn_01x04_Shielded
Connections:
- wire segments 97 -> 96
- no-connect marks 8 -> 13
Other:
- note added: "RS232 Transreceiver\n\n"
- note removed: "RS232"
- moved on the sheet: U3
